File: Hardware/node_sensor/node_sensor.kicad_sch (KiCad schematic)
At the start: 0 parts

Commit message: .
Parts:
- added U1: DevKitESP32, Thao_footprint:kitEsp32Rebuild, symbol MY_SYMBOLS:DevKitESP32
Other:
- title: (none) -> Plant_CPS
Changed lines of the file:
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@@
 	(generator_version "10.0")
 	(paper "A4")
+	(title_block
+		(title "Plant_CPS")
+		(date "2026-05-24")
+		(rev "v1.0")
+	)
+	(symbol
+		(lib_id "MY_SYMBOLS:DevKitESP32")
+		(at 83.82 80.01 0)
+		(unit 1)
+		(body_style 1)
+		(exclude_from_sim no)
+		(in_bom yes)
+		(on_board yes)
+		(in_pos_files yes)
+		(dnp no)
+		(fields_autoplaced yes)
+		(property "Reference" "U1"
+			(at 87.63 48.26 0)
+			(show_name no)
+			(do_not_autoplace no)
+			(effects
+				(font
+					(size 1.27 1.27)
+				)
+			)
+		)
+		(property "Value" "DevKitESP32"
+			(at 87.63 50.8 0)
+			(show_name no)
+			(do_not_autoplace no)
+			(effects
+				(font
+					(size 1.27 1.27)
+				)
+			)
+		)
+		(property "Footprint" "Thao_footprint:kitEsp32Rebuild"
+			(at 88.9 81.915 0)
+			(hide yes)
+			(show_name no)
+			(do_not_autoplace no)
+			(effects
+				(font
+					(size 1.27 1.27)
+				)
+			)
+		)
+		(property "Datasheet" ""
+			(at 83.82 80.01 0)
+			(hide yes)
+			(show_name no)
+			(do_not_autoplace no)
+			(effects
+				(font
+					(size 1.27 1.27)
+				)
+			)
+		)
+		(property "Description" ""
+			(at 83.82 80.01 0)
+			(hide yes)
+			(show_name no)
+			(do_not_autoplace no)
+			(effects
+				(font
+					(size 1.27 1.27)
+				)
+			)
+		)
+		(pin "13"
+		)
+		(pin "36"
+		)
+		(pin "12"
+		)
+		(pin "37"
+		)
+		(pin "29"
+		)
+		(pin "32"
+		)
+		(pin "27"
+		)
+		(pin "26"
+		)
+		(pin "38"
+		)
+		(pin "25"
+		)
+		(pin "11"
+		)
+		(pin "28"
+		)
+		(pin "10"
+		)
+		(pin "9"
+		)
+		(pin "33"
+		)
+		(pin "16"
+		)
+		(pin "34"
+		)
+		(pin "23"
+		)
+		(pin "30"
+		)
+		(pin "35"
+		)
+		(pin "15"
+		)
+		(pin "6"
+		)
+		(pin "24"
+		)
+		(pin "20"
+		)
+		(pin "17"
+		)
+		(pin "4"
+		)
+		(pin "5"
+		)
+		(pin "1"
+		)
+		(pin "2"
+		)
+		(pin "3"
+		)
+		(pin "8"
+		)
+		(pin "21"
+		)
+		(pin "14"
+		)
+		(pin "22"
+		)
+		(pin "31"
+		)
+		(pin "18"
+		)
+		(pin "19"
+		)
+		(pin "7"
+		)
+		(instances
+			(project "node_sensor"
+				(path "/b1f2dde9-9c60-4b08-b31e-edf781363067"
+					(reference "U1")
+					(unit 1)
+				)
+			)
+		)
+	)
 	(sheet_instances
 		(path "/"
